Commit message: work from home

File: my_youbot_twoarm_collab/robots/two_arm_cage.urdf.xacro (robot description, xacro)
@@ -8,8 +8,4 @@
   <!-- misc common stuff? -->
   <xacro:include filename="$(find youbot_description)/urdf/common.xacro" />
-  <!-- youbot base -->
-  <xacro:include filename="$(find youbot_description)/urdf/youbot_base/base.urdf.xacro" />
-  <!-- youbot plate -->
-  <xacro:include filename="$(find youbot_description)/urdf/youbot_plate/plate.urdf.xacro" />
   <!-- youbot arm -->
   <xacro:include filename="$(find youbot_description)/urdf/youbot_arm/arm.urdf.xacro"/>
@@ -34,5 +30,5 @@
     <visual>
       <geometry>
-        <box size="2.0 1.0 0.01"/>
+        <box size="2.0 1.0 0.0"/>
       </geometry>
     </visual>
@@ -44,6 +40,5 @@
   </link>
   <xacro:youbot_arm name="arm" parent="base_link">
-    <!--<origin xyz="0.143 0 0.046" rpy="0 0 0" />-->
-    <origin xyz="1.0 0 0.056" rpy="0 0 0" /> <!-- x offset needs to be further verified -->
+    <origin xyz="0.25 0 0.04225" rpy="0 0 1.57075" />
   </xacro:youbot_arm>
   <xacro:youbot_gripper name="gripper" parent="arm_link_5">
@@ -51,6 +46,5 @@
   </xacro:youbot_gripper>
   <xacro:youbot_arm name="arm_2" parent="base_link">
-    <!--<origin xyz="-0.143 0 0.046" rpy="0 0 0" />-->
-    <origin xyz="-1.0 0 0.056" rpy="0 0 0" />  <!-- x offset needs to be further verified -->
+    <origin xyz="-0.25 0 0.04225" rpy="0 0 1.57075" />
   </xacro:youbot_arm>
   <xacro:youbot_gripper name="gripper_2" parent="arm_2_link_5">

File: youbot_description/urdf/youbot_arm/arm.urdf.xacro (robot description, xacro)
@@ -8,10 +8,8 @@
         <xacro:include filename="$(find youbot_description)/urdf/youbot_arm/limits.urdf.xacro" />
 	<!-- specifies the offset to include the 10mm table flange and the 3.225cm model offset -->
-	<xacro:property name="base_link_zoffset" value="0.04225"/>
 	<xacro:macro name="youbot_arm" params="parent name *origin">
 		<!-- joint between base_link and arm_0_link -->
 		<joint name="${name}_joint_0" type="fixed" >
-			<!--<insert_block name="origin" />-->
-			<origin xyz="0.00 0.0 ${base_link_zoffset}" rpy="0 0 0" />
+			<insert_block name="origin" />
 			<parent link="${parent}" />
 			<child link="${name}_link_0" />
